File: KiCad/ATMegaSpin/ATMegaSpin.kicad_pcb (KiCad board)
At the start: 2 copper layers, 100.2 x 139 mm, 30 parts, among them X1 ED281DT, Y1 ECS-160-18-4X-CKM

Commit message: Adapt tree
Parts:
- moved LED8 47.7 mm to (177.8, 75.7)
- moved LED9 47.7 mm to (177.8, 88.4)
- moved R10 47.7 mm to (177.3, 114.8)
- moved R7 47.7 mm to (182.9, 52.6)
- moved REF** 47.7 mm to (149.1, 131.6)
- moved REF** 47.7 mm to (149.1, 63.0)
- moved B1 47.7 mm to (161.1, 72.1)
- moved LED1 47.7 mm to (147.9, 109.5)
- moved LED10 47.7 mm to (170.2, 103.9)
- moved LED2 47.7 mm to (126.2, 101.9)
- moved LED3 47.7 mm to (120.4, 85.4)
- moved LED4 47.7 mm to (120.4, 72.7)
- moved LED5 47.7 mm to (127.9, 57.8)
- moved LED6 47.7 mm to (150.5, 52.1)
- moved LED7 47.7 mm to (172.0, 59.7)
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
Commit message: Kicad updated
Parts:
- added SW1: MFS101D-6-Z, Library:MFS101D-6-Z_NDC, F.Cu at (160.5, 147.3)
- renumbered REF** to H, REF** to h2
Connections:
- S1 pad 1: Net-(B1-Pad2) -> Net-(S1-Pad1)
- X1 pad 7: Net-(B1-Pad2) -> Net-(S1-Pad1)
Routing:
- net Net-(S1-Pad1): track 0.00 -> 54.0 mm
- net Net-(B1-Pad2): track 85.7 -> 56.4 mm
- net Net-(R8-Pad1): track 107.7 -> 113.9 mm
- net Net-(R10-Pad1): track 56.5 -> 62.1 mm
- net Net-(R5-Pad1): track 124.2 -> 128.9 mm
- net Net-(R3-Pad1): track 99.9 -> 95.2 mm
- net GND: track 272.4 -> 276.3 mm
- net Net-(R2-Pad1): track 79.4 -> 76.1 mm
- net Net-(C2-Pad2): track 28.9 -> 26.1 mm
- net Net-(R9-Pad1): track 88.0 -> 89.0 mm, vias 0 -> 1
- net Net-(R4-Pad1): track 106.9 -> 106.0 mm
