File: KiCad/ATMegaSpin/ATMegaSpin.kicad_pcb (KiCad board)
At the start: 2 copper layers, 100.2 x 139 mm, 31 parts, among them SW1 MFS101D-6-Z, X1 ED281DT, Y1 ECS-160-18-4X-CKM

Commit message: Update files
Connections:
- X1 pad 2: Net-(R1-Pad1) -> unconnected-(X1-Pad2)
- X1 pad 4: unconnected-(X1-Pad4) -> Net-(R1-Pad1)
Routing:
- net Net-(S1-Pad1): track 54.0 -> 43.6 mm
- net GND: track 276.3 -> 284.6 mm
- net Net-(R9-Pad1): track 89.0 -> 96.7 mm, vias 1 -> 0
- net Net-(R8-Pad1): track 113.9 -> 107.7 mm
- net Net-(R5-Pad1): track 128.9 -> 124.2 mm
- net Net-(R3-Pad1): track 95.2 -> 100.0 mm
- net Net-(R2-Pad1): track 76.1 -> 79.0 mm
- net Net-(R1-Pad1): track 50.0 -> 47.9 mm
- net Net-(R4-Pad1): track 106.0 -> 106.9 mm
- net Net-(R10-Pad1): track 62.1 -> 61.6 mm

Commit message: Update 3D View + schematic + GERBER files
Connections:
- LED1 pad 1: GND -> Net-(LED1-Pad1)
- LED1 pad 2: Net-(LED1-Pad2) -> GND
- LED10 pad 1: GND -> Net-(LED10-Pad1)
- LED10 pad 2: Net-(LED10-Pad2) -> GND
- LED2 pad 1: GND -> Net-(LED2-Pad1)
- LED2 pad 2: Net-(LED2-Pad2) -> GND
- LED3 pad 1: GND -> Net-(LED3-Pad1)
- LED3 pad 2: Net-(LED3-Pad2) -> GND
- LED4 pad 1: GND -> Net-(LED4-Pad1)
- LED4 pad 2: Net-(LED4-Pad2) -> GND
- LED5 pad 1: GND -> Net-(LED5-Pad1)
- LED5 pad 2: Net-(LED5-Pad2) -> GND
- LED6 pad 1: GND -> Net-(LED6-Pad1)
- LED6 pad 2: Net-(LED6-Pad2) -> GND
- LED7 pad 1: GND -> Net-(LED7-Pad1)
- LED7 pad 2: Net-(LED7-Pad2) -> GND
- LED8 pad 1: GND -> Net-(LED8-Pad1)
- LED8 pad 2: Net-(LED8-Pad2) -> GND
- LED9 pad 1: GND -> Net-(LED9-Pad1)
- LED9 pad 2: Net-(LED9-Pad2) -> GND
- R1 pad 2: Net-(LED1-Pad2) -> Net-(LED1-Pad1)
- R10 pad 2: Net-(LED10-Pad2) -> Net-(LED10-Pad1)
- R2 pad 2: Net-(LED2-Pad2) -> Net-(LED2-Pad1)
- R3 pad 2: Net-(LED3-Pad2) -> Net-(LED3-Pad1)
- R4 pad 2: Net-(LED4-Pad2) -> Net-(LED4-Pad1)
- R5 pad 2: Net-(LED5-Pad2) -> Net-(LED5-Pad1)
- R6 pad 2: Net-(LED6-Pad2) -> Net-(LED6-Pad1)
- R7 pad 2: Net-(LED7-Pad2) -> Net-(LED7-Pad1)
- R8 pad 2: Net-(LED8-Pad2) -> Net-(LED8-Pad1)
- R9 pad 2: Net-(LED9-Pad2) -> Net-(LED9-Pad1)
Routing:
- net Net-(LED9-Pad1): track 0.00 -> 15.4 mm
- net Net-(LED2-Pad1): track 0.00 -> 14.9 mm
- net Net-(LED7-Pad1): track 0.00 -> 14.9 mm
- net Net-(LED5-Pad1): track 0.00 -> 14.9 mm
- net Net-(LED10-Pad1): track 0.00 -> 14.9 mm
- net Net-(LED8-Pad1): track 0.00 -> 14.9 mm
- net Net-(LED4-Pad1): track 0.00 -> 14.9 mm
- net Net-(LED3-Pad1): track 0.00 -> 14.9 mm
- net Net-(LED6-Pad1): track 0.00 -> 14.9 mm
- net Net-(LED1-Pad1): track 0.00 -> 14.7 mm
- net Net-(LED9-Pad2): track 14.3 -> 0.00 mm
- net Net-(LED2-Pad2): track 13.8 -> 0.00 mm
- net Net-(LED4-Pad2): track 13.8 -> 0.00 mm
- net Net-(LED3-Pad2): track 13.8 -> 0.00 mm
- net Net-(LED6-Pad2): track 13.8 -> 0.00 mm
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